File: pcb/controller/controller.kicad_pcb (KiCad board)
At the start: 2 copper layers, 60 x 70 mm, 35 parts, among them J1 Conn_01x03, J2 Conn_01x03, J3 RELAY_CONN, J4 Remote_header, J5 PWR_IN, J6 MFRC_CONN, J7 Micro_SD_Card, Q1 MMBT3906, Q2 MMBT3906, Q3 IRLL014N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

Commit message: Footprint updates Major restructuring
Parts:
- D1: footprint Diode_SMD:D_1206_3216Metric_Pad1.42x1.75mm_HandSolder -> Diode_SMD:D_SMA-SMB_Universal_Handsoldering
- moved D1 3.35 mm to (61.7, 77.3)
Routing:
- net RELAY+: track 24.2 -> 26.2 mm
- net RELAY-: track 32.7 -> 33.9 mm

Commit message: PCB changes - add GPIO3/4
Parts:
- added J8: Conn_01x03, Connector_JST:JST_XH_B3B-XH-A_1x03_P2.50mm_Vertical, F.Cu at (43.4, 82.8)
- added J9: Conn_01x03, Connector_JST:JST_XH_B3B-XH-A_1x03_P2.50mm_Vertical, F.Cu at (74.8, 83.0)
- added R7: 1K, Resistor_SMD:R_1210_3225Metric_Pad1.30x2.65mm_HandSolder, B.Cu at (75.0, 66.3)
- added R8: R10K, Resistor_SMD:R_1210_3225Metric_Pad1.30x2.65mm_HandSolder, B.Cu at (72.1, 82.2)
- R4, R5, R6: value R -> 91R
- moved R3 10.5 mm to (71.3, 66.2), turned to 90 degrees
- moved D1 2.44 mm to (59.4, 76.4)
- moved JP1 1.88 mm to (77.4, 78.9)
- moved J3 1.83 mm to (64.8, 83.2)
- moved J5 0.81 mm to (54.8, 83.3)
- moved D4 0.46 mm to (82.5, 77.2)
Connections:
- A1 pad 6: unconnected-(A1-GPIO4-Pad6) -> GPIO_ACC3
- A1 pad 7: unconnected-(A1-GPIO5-Pad7) -> GPIO_ACC4
- Q3 pad 1: MOSFET_GATE -> Net-(Q3-G)
- R3 pad 1: MOSFET_GATE -> Net-(Q3-G)
Routing:
- net GPIO_ACC4: track 0.00 -> 91.6 mm, vias 0 -> 1
- net +3V3: track 144.2 -> 208.8 mm
- net GPIO_ACC3: track 0.00 -> 45.0 mm, vias 0 -> 1
- net Net-(Q3-G): track 0.00 -> 13.5 mm
- net RELAY+: track 26.2 -> 37.9 mm
- net MOSFET_GATE: track 26.8 -> 17.4 mm
- net +VDC: track 57.7 -> 55.6 mm
- net ACCESS_DENIED: track 41.2 -> 40.5 mm
- net RELAY-: track 33.9 -> 34.6 mm
- net +5V: track 110.8 -> 110.2 mm
Other:
- board text added: "For 3/5V I/P, bridge JP3 For 7-28VDC I/P, install MP1584 module here"
- board text removed: "For 5V I/P, bridge JP2 For 7-28VDC I/P, install MP1584 module here"
