File: pcb/mains_controller/controller.kicad_pcb (KiCad board)
At the start: 2 copper layers, 60 x 115 mm, 36 parts, among them J1 Conn_01x03, J2 Conn_01x03, J3 Conn_01x03, J4 Conn_01x03, J4 Conn_01x04_Pin, J5 Conn_01x02_Pin, J6 MFRC_CONN, J7 Micro_SD_Card, J8 Conn_01x02_Pin, K2 Relay_SPDT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

Commit message: Update to v1.3
Other:
- board text added: "Access Control Gen2 240V Controller V1.3"
- board text removed: "Access Control Gen2 240V Controller V1.2"
Changed lines of the file:
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@@
 		)
 	)
-	(gr_text "Access Control Gen2\n240V Controller\nV1.2"
+	(gr_text "Access Control Gen2\n240V Controller\nV1.3"
 		(at 65.8 62.6 0)
 		(layer "F.SilkS")

Commit message: Fixes for pcb
Parts:
- removed the J4 at (65.6, 126.2)
- added J9: Conn_01x03, TerminalBlock_MetzConnect:TerminalBlock_MetzConnect_Type073_RT02603HBLU_1x03_P5.08mm_Horizontal, F.Cu at (65.7, 126.1)
- F2: value Fuse -> Thermal fuse
- K2: value Relay_SPDT -> G2RL-1-E-DC5
- moved J3 0.22 mm to (47.4, 126.1)
Connections:
- A1 pad 10: ACCESS_GRANTED -> ACCESS_DENIED
- A1 pad 11: ACCESS_DENIED -> ACCESS_GRANTED
- J5 pad 1: ACCESS_DENIED -> ACCESS_GRANTED
- J8 pad 1: ACCESS_GRANTED -> ACCESS_DENIED
- R5 pad 1: ACCESS_GRANTED -> ACCESS_DENIED
- R6 pad 1: ACCESS_DENIED -> ACCESS_GRANTED
Routing:
- net ACCESS_GRANTED: track 45.2 -> 37.8 mm
- net ACCESS_DENIED: track 37.8 -> 45.2 mm
